File: diagboard-1.00_Kicad/01_DiagBoard1.kicad_pcb (KiCad board)
At the start: 2 copper layers, 84.8 x 80 mm, 34 parts, among them IC1 27C512, IC2 74LS00N, IC3 74273N, IC4 74LS04N, Q1 1.000 MHz

Commit message: Add files via upload
Parts:
- added C1: 100nF, 01_DiagBoard1:C050-024X044, F.Cu at (10.7, 43.8)
- added C2: 100nF, 01_DiagBoard1:C050-024X044, F.Cu at (10.7, 47.3)
- added C3: 100nF, 01_DiagBoard1:C050-024X044, F.Cu at (10.7, 50.7)
- added C4: 1nF, 01_DiagBoard1:C050-024X044, F.Cu at (10.7, 54.1)
- added CLK0: 1MHz, 01_DiagBoard1:1X02, F.Cu at (49.7, 7.75)
- added D1: U57X32, 01_DiagBoard1:U57X32, F.Cu at (3.25, 27.1)
- added D2: U57X32, 01_DiagBoard1:U57X32, F.Cu at (3.25, 32.1)
- added D3: U57X32, 01_DiagBoard1:U57X32, F.Cu at (3.25, 37.0)
- added D4: U57X32, 01_DiagBoard1:U57X32, F.Cu at (3.25, 42.0)
- added D5: U57X32, 01_DiagBoard1:U57X32, F.Cu at (3.25, 46.9)
- added D6: U57X32, 01_DiagBoard1:U57X32, F.Cu at (3.25, 51.9)
- added EXP1: TO ORIC, 01_DiagBoard1:2X17, F.Cu at (21.7, 2.62)
- added IC1: 27C512, 01_DiagBoard1:DIL28, F.Cu at (17.9, 15.2)
- added IC2: 7400N, 01_DiagBoard1:DIL14, F.Cu at (43.0, 30.2)
- added IC3: 74273N, 01_DiagBoard1:DIL20, F.Cu at (20.3, 30.2)
- added IC4: 7404N, 01_DiagBoard1:DIL14, F.Cu at (43.0, 41.5)
- added JP1: A14=0, 01_DiagBoard1:1X02, F.Cu at (49.7, 11.8)
- added JP2: A15=0, 01_DiagBoard1:1X02, F.Cu at (49.7, 15.8)
- added JP4: INHIBIT VIA, 01_DiagBoard1:1X02, F.Cu at (49.7, 19.9)
- added JP5: -VIA SEL, 01_DiagBoard1:1X01, F.Cu at (47.8, 49.0)
- added LPT1: Loopback, 01_DiagBoard1:2X10, F.Cu at (20.3, 39.0)
- added Q1: 1.000 MHz, 01_DiagBoard1:HC18U-V, F.Cu at (39.8, 50.8)
- added R1: 82R, 01_DiagBoard1:0204V, F.Cu at (38.9, 7.20)
- added R10: 1K0, 01_DiagBoard1:0204V, F.Cu at (44.1, 16.0)
- added R11: 10K, 01_DiagBoard1:0204V, F.Cu at (44.1, 18.9)
- added R2: 82R, 01_DiagBoard1:0204V, F.Cu at (38.9, 10.1)
- added R3: 82R, 01_DiagBoard1:0204V, F.Cu at (38.9, 13.1)
- added R4: 82R, 01_DiagBoard1:0204V, F.Cu at (38.9, 16.0)
- added R5: 82R, 01_DiagBoard1:0204V, F.Cu at (38.9, 18.9)
- added R6: 82R, 01_DiagBoard1:0204V, F.Cu at (38.9, 21.8)
- added R7: 2K2, 01_DiagBoard1:0204V, F.Cu at (44.1, 7.20)
- added R8: 2K2, 01_DiagBoard1:0204V, F.Cu at (44.1, 10.1)
- added R9: 1K0, 01_DiagBoard1:0204V, F.Cu at (44.1, 13.1)
- added S1: RESET, 01_DiagBoard1:DT6, F.Cu at (20.3, 48.8)

Commit message: Add files via upload
Parts:
- removed the C1 at (158.7, 119.0)
- removed the C2 at (163.7, 96.1)
- removed the C3 at (139.6, 96.1)
- removed the C4 at (176.4, 130.4)
- removed the CLK0 at (186.6, 124.1)
- removed the D1 at (134.5, 79.6)
- removed the D2 at (130.7, 79.6)
- removed the D3 at (126.9, 79.6)
- removed the D4 at (123.1, 79.6)
- removed the D5 at (119.3, 79.6)
- removed the D6 at (115.5, 79.6)
- removed the EXP1 at (138.3, 139.3)
- removed the IC1 at (137.1, 119.0)
- removed the IC2 at (152.3, 96.1)
- removed the IC3 at (124.4, 96.1)
- removed the IC4 at (180.3, 115.2)
- removed the JP1 at (163.7, 126.6)
- removed the JP2 at (163.7, 111.4)
- removed the JP4 at (149.8, 84.7)
- removed the JP5 at (151.0, 77.1)
- removed the LPT1 at (185.3, 83.4)
- removed the Q1 at (176.4, 136.8)
- removed the R1 at (134.5, 86.0)
- removed the R10 at (179.0, 124.1)
- removed the R11 at (143.4, 78.3)
- removed the R2 at (130.7, 86.0)
- removed the R3 at (126.9, 86.0)
- removed the R4 at (123.1, 86.0)
- removed the R5 at (119.3, 86.0)
- removed the R6 at (115.5, 86.0)
- removed the R7 at (112.9, 110.1)
- removed the R8 at (112.9, 106.3)
- removed the R9 at (173.9, 124.1)
- removed the S1 at (161.2, 80.9)
- R6: value 82R -> 6 x 82R
- moved C4 182.5 mm to (176.5, 130.5)
- moved EXP1 179.4 mm to (138.5, 138.7)
- moved CLK0 179.3 mm to (186.2, 124.0)
- moved R10 172.2 mm to (178.5, 123.8)
- moved LPT1 171.1 mm to (185.5, 83.5), turned to 90 degrees
- moved R9 170.1 mm to (173.2, 123.8)
- moved C1 164.7 mm to (157.0, 119.5), turned to 90 degrees
- moved Q1 161.4 mm to (176.0, 137.5)
- moved C2 160.9 mm to (163.8, 96.8), turned to 90 degrees
- moved JP1 160.7 mm to (163.2, 125.5)
- moved IC1 157.6 mm to (136.0, 119.4)
- moved IC4 155.9 mm to (180.5, 115.0)
- moved JP2 149.8 mm to (163.2, 113.5)
- moved S1 148.8 mm to (166.0, 79.0)
- moved D1 142.8 mm to (135.8, 80.2), turned to 90 degrees
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Connections:
- EXP1 pad 1: /-RST -> unconnected-(EXP1-Pad1)
- EXP1 pad 10: /D0 -> D0
- EXP1 pad 11: /A3 -> A3
- EXP1 pad 12: /D1 -> D1
- EXP1 pad 13: /A0 -> A0
- EXP1 pad 14: /D6 -> D6
- EXP1 pad 15: /A1 -> A1
- EXP1 pad 16: /D3 -> D3
- EXP1 pad 17: /A2 -> A2
- EXP1 pad 18: /D4 -> D4
- EXP1 pad 19: /ADDR:A[0..15] -> D5
- EXP1 pad 2: /-RST -> ~ROMDIS
- EXP1 pad 20: /A4 -> A4
- EXP1 pad 21: /A5 -> A5
- EXP1 pad 22: /ADDR:A[0..15] -> D7
- EXP1 pad 23: /A6 -> A6
- EXP1 pad 24: /A15 -> A15
- EXP1 pad 25: /A7 -> A7
- EXP1 pad 26: /A14 -> A14
- EXP1 pad 27: /A8 -> A8
- EXP1 pad 28: /A13 -> A13
- EXP1 pad 29: /A9 -> A9
- EXP1 pad 3: /-RST -> PH2
- EXP1 pad 30: /A12 -> A12
- EXP1 pad 31: /A10 -> A10
- EXP1 pad 32: /A11 -> A11
- EXP1 pad 4: /-RST -> ~RST
- EXP1 pad 5: /-RST -> unconnected-(EXP1-Pad5)
- EXP1 pad 6: /-RST -> IOCTRL
- EXP1 pad 7: /-RST -> R/~W
- EXP1 pad 8: /-RST -> unconnected-(EXP1-Pad8)
- EXP1 pad 9: /D2 -> D2
- IC1 pad 10: /A0 -> A0
- IC1 pad 11: /D0 -> D0
- IC1 pad 12: /D1 -> D1
- IC1 pad 13: /D2 -> D2
- IC1 pad 15: /D3 -> D3
- IC1 pad 16: /D4 -> D4
- IC1 pad 17: /ADDR:A[0..15] -> D5
- IC1 pad 18: /D6 -> D6
- IC1 pad 19: /ADDR:A[0..15] -> D7
- IC1 pad 2: /A12 -> A12
- IC1 pad 20: /-RST -> ~ROMDIS
- IC1 pad 21: /A10 -> A10
- IC1 pad 23: /A11 -> A11
- IC1 pad 24: /A9 -> A9
- IC1 pad 25: /A8 -> A8
- IC1 pad 26: /A13 -> A13
- IC1 pad 3: /A7 -> A7
- IC1 pad 4: /A6 -> A6
- IC1 pad 5: /A5 -> A5
- IC1 pad 6: /A4 -> A4
- IC1 pad 7: /A3 -> A3
- IC1 pad 8: /A2 -> A2
- IC1 pad 9: /A1 -> A1
- IC2 pad 1: /A15 -> A15
- IC2 pad 2: /A14 -> A14
- IC2 pad 3: /-RST -> ~ROMDIS
- IC2 pad 4: /-RST -> R/~W
- IC2 pad 5: /-RST -> PH2
- IC3 pad 1: /-RST -> ~RST
- IC3 pad 13: /A4 -> A4
- IC3 pad 14: /A5 -> A5
- IC3 pad 17: /A6 -> A6
- IC3 pad 18: /A7 -> A7
- IC3 pad 3: /A0 -> A0
- IC3 pad 4: /A1 -> A1
- IC3 pad 7: /A2 -> A2
- IC3 pad 8: /A3 -> A3
- JP4 pad 1: /-RST -> IOCTRL
- JP5 pad 1: /-RST -> -IO
- R11 pad 1: /-RST -> -IO
- S1 pad 3: /-RST -> ~RST
- S1 pad 4: /-RST -> ~RST
Routing:
- net -RST: track 155.9 -> 0.00 mm
- net ~RST: track 0.00 -> 113.7 mm, vias 0 -> 1
- net -IO: track 89.8 -> 9.84 mm, vias 1 -> 0
- net Net-(IC1A-A15): track 0.00 -> 75.7 mm
- net N$3: track 74.1 -> 0.00 mm
- net ~ROMDIS: track 0.00 -> 73.6 mm, vias 0 -> 1
- net -ROMDIS: track 73.0 -> 0.00 mm
- net VCC: track 269.3 -> 201.2 mm
- net N$2: track 65.1 -> 0.00 mm
- net R/~W: track 0.00 -> 64.4 mm, vias 0 -> 1
- net Net-(IC1A-A14): track 0.00 -> 55.7 mm
- net A14: track 92.6 -> 38.0 mm, vias 1 -> 0
- net GND: track 268.7 -> 216.6 mm
- net LOW=PH2+READ: track 46.3 -> 0.00 mm
- net /LOW=PH2+READ: track 0.00 -> 45.4 mm
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- added copper zone on B.Cu, net GND
- added copper zone on F.Cu, net GND
